Commit message: Add COAL-backed SE(3) collision planning

File: etc/URDF-for-gazebo/urdf/HDJQR-0102-0055.SLDASM.urdf (robot description, URDF)
Before this commit: robot HDJQR-0102-0055.SLDASM, 10 links, 9 joints
Links:
- link base_link: geometry collision box size=0.49607 0.23920 0.22884; collision cylinder length=0.05980 radius=0.19934
- link l1: geometry visual mesh filename=package://HDJQR-0102-0055.SLDASM/meshes/l1.STL
- link l2: geometry visual mesh filename=package://HDJQR-0102-0055.SLDASM/meshes/l2.STL
- link r1: geometry visual mesh filename=package://HDJQR-0102-0055.SLDASM/meshes/r1.STL
- link r2: geometry visual mesh filename=package://HDJQR-0102-0055.SLDASM/meshes/r2.STL
- link xy1: geometry visual mesh filename=package://HDJQR-0102-0055.SLDASM/meshes/xy1.STL
- link xy2: geometry visual mesh filename=package://HDJQR-0102-0055.SLDASM/meshes/xy2.STL
- link xy3: geometry visual mesh filename=package://HDJQR-0102-0055.SLDASM/meshes/xy3.STL
- link xy4: geometry visual mesh filename=package://HDJQR-0102-0055.SLDASM/meshes/xy4.STL
- link xy5: geometry visual mesh filename=package://HDJQR-0102-0055.SLDASM/meshes/xy5.STL
